File: Amp/otl.brd (EAGLE design)
At the start: 154.9 x 68.6 mm, 59 parts, among them X1 MOUNT-PAD2.0, X10 MOUNT-PAD2.0, X11 MOUNT-PAD2.0, X2 MOUNT-PAD2.0, X3 MOUNT-PAD2.0, X4 MOUNT-PAD2.0, X5 MOUNT-PAD2.0, X6 MOUNT-PAD2.0, X7 MOUNT-PAD2.0, X8 MOUNT-PAD2.0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

Commit message: Power buses separated
Connections:
- removed net HT: R10.P$2, R17.P$2, R19.P$2, R22.P$2, R24.P$2, R3.P$2, R5.P$2, R8.P$2, X1.P$1, X11.P$1
- new net HT_L: R10.P$2, R3.P$2, R5.P$2, R8.P$2, X11.P$1
- new net HT_R: R17.P$2, R19.P$2, R22.P$2, R24.P$2, X1.P$1
Routing:
- net HT: track 62.8 -> 0.00 mm
- net HT_L: track 0.00 -> 31.4 mm
- net HT_R: track 0.00 -> 31.4 mm
Changed lines of the file:
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@@
 <wire x1="57.15" y1="12.7" x2="54.61" y2="12.7" width="1.778" layer="1"/>
-</signal>
-<signal name="HT">
-<contactref element="R8" pad="P$2"/>
-<contactref element="R10" pad="P$2"/>
-<contactref element="R3" pad="P$2"/>
-<contactref element="R22" pad="P$2"/>
-<contactref element="R24" pad="P$2"/>
-<contactref element="R17" pad="P$2"/>
-<contactref element="X1" pad="P$1"/>
-<wire x1="105.41" y1="55.88" x2="105.41" y2="59.055" width="2.54" layer="16"/>
-<wire x1="105.41" y1="59.055" x2="105.41" y2="62.23" width="2.54" layer="16"/>
-<wire x1="105.41" y1="12.7" x2="105.41" y2="9.525" width="2.54" layer="16"/>
-<wire x1="105.41" y1="9.525" x2="105.41" y2="6.35" width="2.54" layer="16"/>
-<wire x1="123.19" y1="59.69" x2="122.555" y2="59.055" width="2.54" layer="16" curve="-90"/>
-<wire x1="122.555" y1="59.055" x2="109.22" y2="59.055" width="2.54" layer="16"/>
-<wire x1="109.22" y1="59.055" x2="105.41" y2="59.055" width="2.54" layer="16"/>
-<wire x1="123.19" y1="8.89" x2="122.555" y2="9.525" width="2.54" layer="16" curve="90"/>
-<wire x1="122.555" y1="9.525" x2="109.22" y2="9.525" width="2.54" layer="16"/>
-<contactref element="R5" pad="P$2"/>
-<contactref element="R19" pad="P$2"/>
-<wire x1="109.22" y1="9.525" x2="105.41" y2="9.525" width="2.54" layer="16"/>
-<wire x1="109.22" y1="6.35" x2="109.22" y2="9.525" width="2.54" layer="16"/>
-<wire x1="109.22" y1="62.23" x2="109.22" y2="59.055" width="2.54" layer="16"/>
-<contactref element="X11" pad="P$1"/>
-<wire x1="123.19" y1="5.08" x2="123.19" y2="8.89" width="2.54" layer="16"/>
-<wire x1="123.19" y1="63.5" x2="123.19" y2="59.69" width="2.54" layer="16"/>
-<wire x1="105.41" y1="12.7" x2="105.41" y2="55.88" width="0" layer="19" extent="1-1"/>
 </signal>
 <signal name="N$5">
@@
 <wire x1="88.9" y1="43.307" x2="88.9" y2="52.07" width="1.778" layer="1"/>
 </signal>
+<signal name="HT_L">
+<contactref element="R3" pad="P$2"/>
+<contactref element="R5" pad="P$2"/>
+<contactref element="R8" pad="P$2"/>
+<contactref element="R10" pad="P$2"/>
+<wire x1="105.41" y1="12.7" x2="105.41" y2="9.525" width="2.54" layer="16"/>
+<wire x1="105.41" y1="9.525" x2="105.41" y2="6.35" width="2.54" layer="16"/>
+<wire x1="122.555" y1="9.525" x2="109.22" y2="9.525" width="2.54" layer="16"/>
+<wire x1="109.22" y1="9.525" x2="105.41" y2="9.525" width="2.54" layer="16"/>
+<contactref element="X11" pad="P$1"/>
+<wire x1="109.22" y1="6.35" x2="109.22" y2="9.525" width="2.54" layer="16"/>
+<wire x1="122.555" y1="9.525" x2="123.19" y2="8.89" width="2.54" layer="16" curve="-90"/>
+<wire x1="123.19" y1="8.89" x2="123.19" y2="5.08" width="2.54" layer="16"/>
+</signal>
+<signal name="HT_R">
+<contactref element="R17" pad="P$2"/>
+<contactref element="R19" pad="P$2"/>
+<contactref element="R22" pad="P$2"/>
+<contactref element="R24" pad="P$2"/>
+<wire x1="105.41" y1="55.88" x2="105.41" y2="59.055" width="2.54" layer="16"/>
+<wire x1="105.41" y1="59.055" x2="105.41" y2="62.23" width="2.54" layer="16"/>
+<wire x1="122.555" y1="59.055" x2="109.22" y2="59.055" width="2.54" layer="16"/>
+<wire x1="109.22" y1="59.055" x2="105.41" y2="59.055" width="2.54" layer="16"/>
+<contactref element="X1" pad="P$1"/>
+<wire x1="122.555" y1="59.055" x2="123.19" y2="59.69" width="2.54" layer="16" curve="90"/>
+<wire x1="123.19" y1="59.69" x2="123.19" y2="63.5" width="2.54" layer="16"/>
+<wire x1="109.22" y1="62.23" x2="109.22" y2="59.055" width="2.54" layer="16"/>
+</signal>
 </signals>
